File: Cricuit/accelerometers.kicad_sch (KiCad schematic)
At the start: 10 parts, among them U15 MPU-6050, U16 MPU-6050, U17 MPU-6050, U18 MPU-6050, U19 MPU-6050, U20 MPU-6050, U21 MPU-6050, U22 MPU-6050, U23 MPU-6050, U24 MPU-6050

Commit message: Added electromagnet subsheet
Now we have GPIO pin assignments for all components
Other:
- company: (none) -> CMD_SAT
- title: (none) -> MPU-6050 I2C Bus Wiring
Changed lines of the file:
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@@
 (kicad_sch (version 20230121) (generator eeschema)
   (paper "A4")
+  (title_block
+    (title "MPU-6050 I2C Bus Wiring")
+    (date "2024-02-23")
+    (company "CMD_SAT")
+  )
   (junction (at 72.39 57.15) (diameter 0) (color 0 0 0 0)
   )
